File: PA-2W for modifyed sxceiver/PA-2W for modifyed sxceiver.kicad_pcb (KiCad board)
At the start: 2 copper layers, 61.5 x 32.2 mm, 33 parts, among them J1 SMA_RF IN, J2 SMA_RF OUT, J3 5Vcc input, U2 TQP7M9106

Commit message: Add files via upload
Parts:
- removed FL1: LFCN-490, Filter:Filter_Mini-Circuits_FV1206
- added REF**: OSHW-Logo_5.7x6mm_SilkScreen, Symbol:OSHW-Logo_5.7x6mm_SilkScreen, F.Cu at (135.0, 115.8)
- moved J2 3.50 mm to (161.9, 108.8)
Connections:
- C12 pad 2: Net-(FL1-IN) -> Net-(J2-In)
- J2 pad 1: Net-(FL1-OUT) -> Net-(J2-In)
Routing:
- net Net-(J2-In): track 0.00 -> 5.98 mm
- net Net-(FL1-OUT): track 4.16 -> 0.00 mm
- net Net-(FL1-IN): track 2.23 -> 0.00 mm
- net GND: track 18.5 -> 16.4 mm, vias 10 -> 21
Other:
- board size 61.5 x 32.2 mm -> 58.2 x 32.2 mm
- board text added: "V1.1"
- board text added: "Z32IT"
