File: PA-2W for sxceiver with PA/PA-2W for sxceiver with PA.kicad_pcb (KiCad board)
At the start: 2 copper layers, 65.5 x 30.8 mm, 33 parts, among them J1 SMA_RF IN, J2 SMA_RF OUT, J3 5Vcc input, U1 TQP7M9106

Commit message: Add files via upload
Parts:
- removed H6: MountingHole, MountingHole:MountingHole_2.2mm_M2_DIN965_Pad
- removed the REF** at (161.0, 94.8)
- added H3: MountingHole_2.7mm_M2.5_Pad_Via, MountingHole:MountingHole_2.7mm_M2.5_Pad_Via, F.Cu at (149.2, 115.5)
- added REF**: OSHW-Logo2_7.3x6mm_Copper, Symbol:OSHW-Logo2_7.3x6mm_Copper, F.Cu at (161.8, 94.8)
- C6: footprint Capacitor_SMD:C_0805_2012Metric -> Capacitor_SMD:C_0603_1608Metric_Pad1.08x0.95mm_HandSolder
- H1, H2, H4: value MountingHole -> MountingHole_2.7mm_M2.5_Pad_Via; footprint MountingHole:MountingHole_2.2mm_M2_DIN965_Pad -> MountingHole:MountingHole_2.7mm_M2.5_Pad_Via
- moved H4 33.4 mm to (125.0, 115.5)
- moved H2 30.1 mm to (149.2, 100.0)
- moved H1 1.60 mm to (125.0, 100.0)
- moved C6 0.25 mm to (122.8, 94.0)
Connections:
- C9 pad 1: /RF_OUT/VCC -> Net-(C10-Pad1)
- H1 pad 1: (no net) -> GND
- L3 pad 2: /RF_OUT/VCC -> Net-(C10-Pad1)
- L4 pad 1: /RF_OUT/VCC -> Net-(C10-Pad1)
Routing:
- net GND: vias 28 -> 26
Other:
- board text added: "PA 2W"
- board text removed: "V1.2"
