File: PA-2W for sxceiver with PA/PA-2W for sxceiver with PA.kicad_sch (KiCad schematic)
At the start: 34 parts, among them J1 SMA_RF IN, J2 SMA_RF OUT, J3 5Vcc input, U1 TQP7M9106

Commit message: Add files via upload
Parts:
- removed H5, H6: MountingHole, MountingHole:MountingHole_2.2mm_M2_DIN965_Pad, symbol Mechanical:MountingHole
- C6: footprint Capacitor_SMD:C_0805_2012Metric -> Capacitor_SMD:C_0603_1608Metric_Pad1.08x0.95mm_HandSolder
- H1, H2, H3, H4: footprint MountingHole:MountingHole_2.2mm_M2_DIN965_Pad -> MountingHole:MountingHole_2.7mm_Pad_Via
