File: PA-2W for -HS- with PA/PA-2W for -HS- with PA.kicad_sch (KiCad schematic)
At the start: 34 parts, among them J1 SMA_RF IN, J2 SMA_RF OUT, J3 5Vcc input, U2 TQP7M9106

Commit message: Add files via upload
Parts:
- removed J1: SMA_RF IN, PCM_SparkFun-Connector:SMA_Edge_SMD, symbol Connector:Conn_Coaxial
- removed J2: SMA_RF OUT, PCM_SparkFun-Connector:SMA_Edge_SMD, symbol Connector:Conn_Coaxial
- added J1: RF-in, Connector_Coaxial:SMA_Amphenol_132289_EdgeMount, symbol PCM_SparkFun-RF:SMA_EdgeMount_6.3mm
- added J2: RF-out, Connector_Coaxial:SMA_Amphenol_132289_EdgeMount, symbol PCM_SparkFun-RF:SMA_EdgeMount_6.3mm
Connections:
- net GND: now also J1.2 (Ext), J2.2 (Ext)
- net at FL1.3 (OUT): now also J2.1 (In)
- net at C4.2: now also J1.1 (In)
Changed lines of the file:
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@@
 	(title_block
 		(title "PA 2W for HS wit PA onboard")
-		(date "2026-04-11")
-		(rev "V2.3")
+		(date "2026-04-12")
+		(rev "V2.4")
 		(company "Z32IT")
 	)
@@
 	)
 	(symbol
+		(lib_id "PCM_SparkFun-RF:SMA_EdgeMount_6.3mm")
+		(at 260.35 114.3 0)
+		(unit 1)
+		(exclude_from_sim no)
+		(in_bom yes)
+		(on_board yes)
+		(dnp no)
+		(property "Reference" "J2"
+			(at 264.16 115.8633 0)
+			(effects
+				(font
+					(size 1.27 1.27)
+				)
+				(justify left)
+			)
+		)
+		(property "Value" "RF-out"
+			(at 264.16 113.3233 0)
+			(effects
+				(font
+					(size 1.27 1.27)
+				)
+				(justify left)
+			)
+		)
+		(property "Footprint" "Connector_Coaxial:SMA_Amphenol_132289_EdgeMount"
+			(at 260.35 124.46 0)
+			(effects
+				(font
+					(size 1.27 1.27)
+				)
+				(hide yes)
+			)
+		)
+		(property "Datasheet" "https://cdn.sparkfun.com/assets/4/1/2/2/0/SMA-Connector.pdf"
+			(at 260.35 127 0)
+			(effects
+				(font
+					(size 1.27 1.27)
+				)
+				(hide yes)
+			)
+		)
+		(property "Description" "Not for new designs. Use 8mm variant. SMA PCB Edge Mount connector"
+			(at 260.35 129.54 0)
+			(effects
+				(font
+					(size 1.27 1.27)
+				)
+				(hide yes)
+			)
+		)
+		(property "PROD_ID" "CONN-08289"
+			(at 260.35 121.92 0)
+			(effects
+				(font
+					(size 1.27 1.27)
+				)
+				(hide yes)
+			)
+		)
+		(pin "1"
+		)
+		(pin "2"
+		)
+		(instances
+			(project "PA-2W for -HS- with PA"
+				(path "/9e841ece-bd19-4cb2-9a9c-7f7db9f00b2a"
+					(reference "J2")
+					(unit 1)
+				)
+			)
+		)
+	)
+	(symbol
 		(lib_id "RF_Filter:LFCN-490")
 		(at 240.03 114.3 0)
@@
 	)
 	(symbol
-		(lib_id "Connector:Conn_Coaxial")
-		(at 260.35 114.3 0)
-		(unit 1)
-		(exclude_from_sim no)
-		(in_bom yes)
-		(on_board yes)
-		(dnp no)
-		(fields_autoplaced yes)
-		(property "Reference" "J2"
-			(at 264.16 113.3231 0)
-			(effects
-				(font
-					(size 1.27 1.27)
-				)
-				(justify left)
-			)
-		)
-		(property "Value" "SMA_RF OUT"
-			(at 264.16 115.8631 0)
-			(effects
-				(font
-					(size 1.27 1.27)
-				)
-				(justify left)
-			)
-		)
-		(property "Footprint" "PCM_SparkFun-Connector:SMA_Edge_SMD"
-			(at 260.35 114.3 0)
-			(effects
-				(font
-					(size 1.27 1.27)
-				)
-				(hide yes)
-			)
-		)
-		(property "Datasheet" "~"
-			(at 260.35 114.3 0)
-			(effects
-				(font
-					(size 1.27 1.27)
-				)
-				(hide yes)
-			)
-		)
-		(property "Description" "coaxial connector (BNC, SMA, SMB, SMC, Cinch/RCA, LEMO, ...)"
-			(at 260.35 114.3 0)
-			(effects
-				(font
-					(size 1.27 1.27)
-				)
-				(hide yes)
-			)
-		)
-		(property "Manufacturer " "RF Solutions"
-			(at 260.35 114.3 0)
-			(effects
-				(font
-					(size 1.27 1.27)
-				)
-				(hide yes)
-			)
-		)
-		(property "Manufacturer Product Number" "CON-SMA-EDGE-S"
-			(at 260.35 114.3 0)
-			(effects
-				(font
-					(size 1.27 1.27)
-				)
-				(hide yes)
-			)
-		)
-		(property "DigiKey Part Number" "CON-SMA-EDGE-S-ND"
-			(at 260.35 114.3 0)
-			(effects
-				(font
-					(size 1.27 1.27)
-				)
-				(hide yes)
-			)
-		)
-		(pin "2"
-		)
-		(pin "1"
-		)
-		(instances
-			(project "LNA-2W"
-				(path "/9e841ece-bd19-4cb2-9a9c-7f7db9f00b2a"
-					(reference "J2")
-					(unit 1)
-				)
-			)
-		)
-	)
-	(symbol
-		(lib_id "Connector:Conn_Coaxial")
+		(lib_id "PCM_SparkFun-RF:SMA_EdgeMount_6.3mm")
 		(at 82.55 115.57 0)
 		(mirror y)
@@
 			)
 		)
-		(property "Value" "SMA_RF IN"
+		(property "Value" "RF-in"
 			(at 78.74 114.5933 0)
 			(effects
@@
 			)
 		)
-		(property "Footprint" "PCM_SparkFun-Connector:SMA_Edge_SMD"
-			(at 82.55 115.57 0)
-			(effects
-				(font
-					(size 1.27 1.27)
-				)
-				(hide yes)
-			)
-		)
-		(property "Datasheet" "~"
-			(at 82.55 115.57 0)
+		(property "Footprint" "Connector_Coaxial:SMA_Amphenol_132289_EdgeMount"
+			(at 82.55 125.73 0)
 			(effects
 				(font
@@
 			)
 		)
-		(property "Description" "coaxial connector (BNC, SMA, SMB, SMC, Cinch/RCA, LEMO, ...)"
-			(at 82.55 115.57 0)
+		(property "Datasheet" "https://cdn.sparkfun.com/assets/4/1/2/2/0/SMA-Connector.pdf"
+			(at 82.55 128.27 0)
 			(effects
 				(font
@@
 			)
 		)
-		(property "Manufacturer" "RF Solutions"
-			(at 82.55 115.57 0)
+		(property "Description" "Not for new designs. Use 8mm variant. SMA PCB Edge Mount connector"
+			(at 82.55 130.81 0)
 			(effects
 				(font
@@
 			)
 		)
-		(property "Manufacturer Product Number" "CON-SMA-EDGE-S"
-			(at 82.55 115.57 0)
+		(property "PROD_ID" "CONN-08289"
+			(at 82.55 123.19 0)
 			(effects
 				(font
@@
 			)
 		)
-		(property "DigiKey Part Number" "CON-SMA-EDGE-S-ND"
-			(at 82.55 115.57 0)
-			(effects
-				(font
-					(size 1.27 1.27)
-				)
-				(hide yes)
-			)
+		(pin "1"
 		)
 		(pin "2"
 		)
-		(pin "1"
-		)
 		(instances
-			(project ""
+			(project "PA-2W for -HS- with PA"
 				(path "/9e841ece-bd19-4cb2-9a9c-7f7db9f00b2a"
 					(reference "J1")

Commit message: Add files via upload
Parts:
- added R5: 10R, Resistor_SMD:R_0603_1608Metric, symbol Device:R_Small
- added R6: 10R, Resistor_SMD:R_0603_1608Metri, symbol Device:R_Small
- R3, R4: value 280R -> 270R
Connections:
- net at C13.1, C14.2, C15.1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: now also R5.1, R6.1; no longer R3.1, R4.1
- new net: R4.1, R6.2
- new net: R3.1, R5.2
