File: PA-2W for -HS- with PA/PA-2W for -HS- with PA.kicad_pcb (KiCad board)
At the start: 2 copper layers, 74 x 30.8 mm, 33 parts, among them J1 SMA_RF IN, J2 SMA_RF OUT, J3 5Vcc input, U2 TQP7M9106

Commit message: Add files via upload
Other:
- board size 74 x 30.8 mm -> 73.5 x 30.8 mm
Changed lines of the file:
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@@
 	(gr_line
 		(start 99.75 88.75)
-		(end 173.75 88.75)
+		(end 173.25 88.75)
 		(stroke
 			(width 0.05)
@@
 	)
 	(gr_line
-		(start 99.75 119.375)
-		(end 99.75 104.625)
+		(start 99.75 119.5)
+		(end 99.75 104.5)
 		(stroke
 			(width 0.05)
@@
 	)
 	(gr_line
-		(start 173.75 119.5)
+		(start 173.25 119.5)
 		(end 99.75 119.5)
 		(stroke
@@
 	)
 	(gr_line
-		(start 173.75 88.75)
-		(end 173.75 119.5)
+		(start 173.25 88.75)
+		(end 173.25 119.5)
 		(stroke
 			(width 0.05)
@@
 		(polygon
 			(pts
-				(xy 115 110.75) (xy 120 110.75) (xy 120 110.25) (xy 173.75 110.25) (xy 173.75 119.5) (xy 115 119.5)
+				(xy 115 110.75) (xy 120 110.75) (xy 120 110.25) (xy 173.25 110.25) (xy 173.25 119.5) (xy 115 119.5)
 			)
 		)
@@
 		(polygon
 			(pts
-				(xy 143.5 107) (xy 143.5 88.75) (xy 173.75 88.75) (xy 173.75 107)
+				(xy 143.5 107) (xy 143.5 88.75) (xy 173.25 88.75) (xy 173.25 107)
 			)
 		)
@@
 		(polygon
 			(pts
-				(xy 99.75 88.75) (xy 173.75 88.75) (xy 173.75 119.5) (xy 99.75 119.5)
-			)
-		)
+				(xy 99.75 88.75) (xy 173.25 88.75) (xy 173.25 119.5) (xy 99.75 119.5)
+			)
+		)

Commit message: Add files via upload
Parts:
- H1, H2, H4, H6: footprint MountingHole:MountingHole_2.7mm_M2.5_Pad_Via -> MountingHole:MountingHole_2.2mm_M2_DIN965_Pad
- J1: value SMA_RF IN -> RF-in; footprint PCM_SparkFun-Connector:SMA_Edge_SMD -> Connector_Coaxial:SMA_Amphenol_132289_EdgeMount
- J2: value SMA_RF OUT -> RF-out; footprint PCM_SparkFun-Connector:SMA_Edge_SMD -> Connector_Coaxial:SMA_Amphenol_132289_EdgeMount
- moved J2 3.86 mm to (169.4, 108.8), turned to 0 degrees
- moved J1 3.60 mm to (103.5, 109.0), turned to 180 degrees
- turned C4 to 180 degrees
Connections:
- C4 pad 1: Net-(J1-In) -> Net-(C4-Pad1)
- C4 pad 2: Net-(C4-Pad1) -> Net-(J1-In)
- C5 pad 1: Net-(C4-Pad1) -> Net-(C5-Pad1)
- C5 pad 2: Net-(C5-Pad1) -> Net-(C4-Pad1)
Routing:
- net Net-(J1-In): track 3.76 -> 8.72 mm
- net Net-(FL1-OUT): track 3.55 -> 8.41 mm
Other:
- board size 73.5 x 30.8 mm -> 72 x 30.8 mm

Commit message: Add files via upload
Parts:
- moved REF** 5.01 mm to (158.2, 95.0)
- moved J2 4.15 mm to (165.2, 108.5)
- moved C11 3.00 mm to (149.5, 109.8)
- moved L4 2.50 mm to (145.8, 108.8)
- moved C10 2.25 mm to (143.0, 109.8)
- moved C12 2.00 mm to (153.2, 108.8)
- moved FL1 2.00 mm to (158.0, 108.7)
- moved C7 1.75 mm to (130.8, 109.8)
Connections:
- U2 pad 27: (no net) -> GND
- U2 pad 28: (no net) -> GND
- U2 pad 29: (no net) -> GND
- U2 pad 30: (no net) -> GND
- U2 pad 31: (no net) -> GND
- U2 pad 32: (no net) -> GND
- U2 pad 33: (no net) -> GND
- U2 pad 34: (no net) -> GND
- U2 pad 35: (no net) -> GND
- U2 pad 36: (no net) -> GND
- U2 pad 37: (no net) -> GND
- U2 pad 38: (no net) -> GND
- U2 pad 39: (no net) -> GND
- U2 pad 40: (no net) -> GND
- U2 pad 41: (no net) -> GND
- U2 pad 42: (no net) -> GND
Routing:
- net /RF_OUT/VCC: track 13.9 -> 10.3 mm
- net Net-(FL1-OUT): track 8.41 -> 5.70 mm
- net GND: track 17.1 -> 16.0 mm
- net Net-(C11-Pad2): track 5.44 -> 5.94 mm
- added copper zone on F.Cu, net /RF_IN
- added copper zone on F.Cu, net /RF_OUT/VCC
Other:
- board size 72 x 30.8 mm -> 67.5 x 30.8 mm

Commit message: Add files via upload
Parts:
- added R5: 10R, Resistor_SMD:R_0603_1608Metric, F.Cu at (138.8, 94.2)
- added R6: 10R, Resistor_SMD:R_0603_1608Metric, F.Cu at (130.8, 94.2)
- H1, H2, H4, H6: footprint MountingHole:MountingHole_2.2mm_M2_DIN965_Pad -> MountingHole:MountingHole_2.7mm_M2.5_Pad_Via
- R3, R4: value 280R -> 270R
- moved R3 1.00 mm to (138.8, 97.8)
- moved R4 1.00 mm to (130.8, 97.8)
- moved J2 0.35 mm to (165.0, 108.8)
Connections:
- R3 pad 1: Net-(C13-Pad1) -> Net-(R3-Pad1)
- R4 pad 1: Net-(C13-Pad1) -> Net-(R4-Pad1)
Routing:
- net GND: track 16.0 -> 7.13 mm, vias 38 -> 44
- net Net-(C13-Pad1): track 41.8 -> 36.4 mm
- net Net-(R4-Pad1): track 0.00 -> 1.85 mm
- net Net-(R3-Pad1): track 0.00 -> 1.85 mm
- net Net-(U2-VBIAS): track 11.8 -> 10.6 mm
- net Net-(C8-Pad1): track 4.64 -> 3.64 mm
Other:
- board size 67.5 x 30.8 mm -> 67.2 x 30.8 mm

Commit message: Add files via upload
Parts:
- moved C12 3.25 mm to (156.5, 108.8)
- moved FL1 2.75 mm to (160.8, 108.7)
- moved J2 2.00 mm to (167.0, 108.8)
- moved C16 0.25 mm to (143.5, 93.2)
- turned C5 to 180 degrees
Routing:
- net Net-(C11-Pad2): track 5.94 -> 9.19 mm
- net Net-(FL1-OUT): track 5.70 -> 4.91 mm
- net Net-(FL1-IN): track 2.48 -> 1.88 mm
Other:
- board size 67.2 x 30.8 mm -> 69.2 x 30.8 mm
Changed lines of the file:
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@@
 	(footprint "Capacitor_SMD:C_0603_1608Metric"
 		(layer "F.Cu")
-		(at 118 109.775)
+		(at 118 109.775 180)
 		(descr "Capacitor SMD 0603 (1608 Metric), square (rectangular) end terminal, IPC_7351 nominal, (Body size source: IPC-SM-782 page 76, https://www.pcb-3d.com/wordpress/wp-content/uploads/ipc-sm-782a_amendment_1_and_2.pdf), generated with kicad-footprint-generator")
 		(tags "capacitor")
 		(property "Reference" "C5"
-			(at 0 1.475 0)
+			(at 0 -1.475 0)
 			(layer "F.SilkS")
 			(effects
@@
 		)
 		(property "Datasheet" "~"
-			(at 0 0 0)
+			(at 0 0 180)
 			(unlocked yes)
 			(layer "F.Fab")
@@
 		)
 		(property "Description" ""
-			(at 0 0 0)
+			(at 0 0 180)
 			(unlocked yes)
 			(layer "F.Fab")
@@
 		)
 		(property "Manufacturer" "YAGEO"
-			(at 0 0 0)
+			(at 0 0 180)
 			(unlocked yes)
 			(layer "F.Fab")
@@
 		)
 		(property "Manufacturer Product Number" "CC0603FRNPO9BN101"
-			(at 0 0 0)
+			(at 0 0 180)
 			(unlocked yes)
 			(layer "F.Fab")
@@
 		)
 		(property "DigiKey Part Number" "311-3599-1-ND"
-			(at 0 0 0)
+			(at 0 0 180)
 			(unlocked yes)
 			(layer "F.Fab")
@@
 		(attr smd)
 		(fp_line
-			(start -0.14058 -0.51)
-			(end 0.14058 -0.51)
+			(start -0.14058 0.51)
+			(end 0.14058 0.51)
 			(stroke
 				(width 0.12)
@@
 		)
 		(fp_line
-			(start -0.14058 0.51)
-			(end 0.14058 0.51)
+			(start -0.14058 -0.51)
+			(end 0.14058 -0.51)
 			(stroke
 				(width 0.12)
@@
 		)
 		(fp_line
-			(start -1.48 -0.73)
-			(end 1.48 -0.73)
+			(start 1.48 0.73)
+			(end -1.48 0.73)
 			(stroke
 				(width 0.05)
@@
 		)
 		(fp_line
-			(start -1.48 0.73)
-			(end -1.48 -0.73)
+			(start 1.48 -0.73)
+			(end 1.48 0.73)
 			(stroke
 				(width 0.05)
@@
 		)
 		(fp_line
-			(start 1.48 -0.73)
-			(end 1.48 0.73)
+			(start -1.48 0.73)
+			(end -1.48 -0.73)
 			(stroke
 				(width 0.05)
@@
 		)
 		(fp_line
-			(start 1.48 0.73)
-			(end -1.48 0.73)
+			(start -1.48 -0.73)
+			(end 1.48 -0.73)
 			(stroke
 				(width 0.05)
@@
 		)
 		(fp_line
-			(start -0.8 -0.4)
-			(end 0.8 -0.4)
+			(start 0.8 0.4)
+			(end -0.8 0.4)
 			(stroke
 				(width 0.1)
@@
 		)
 		(fp_line
-			(start -0.8 0.4)
-			(end -0.8 -0.4)
+			(start 0.8 -0.4)
+			(end 0.8 0.4)
 			(stroke
 				(width 0.1)
@@
 		)
 		(fp_line
-			(start 0.8 -0.4)
-			(end 0.8 0.4)
+			(start -0.8 0.4)
+			(end -0.8 -0.4)
 			(stroke
 				(width 0.1)
@@
 		)
 		(fp_line
-			(start 0.8 0.4)
-			(end -0.8 0.4)
+			(start -0.8 -0.4)
+			(end 0.8 -0.4)
 			(stroke
 				(width 0.1)
@@
 		)
 		(pad "1" smd roundrect
-			(at -0.775 0)
+			(at -0.775 0 180)
 			(size 0.9 0.95)
 			(layers "F.Cu" "F.Mask" "F.Paste")
@@
 		)
 		(pad "2" smd roundrect
-			(at 0.775 0)
+			(at 0.775 0 180)
 			(size 0.9 0.95)
 			(layers "F.Cu" "F.Mask" "F.Paste")
@@
 	(footprint "Connector_Coaxial:SMA_Amphenol_132289_EdgeMount"
 		(layer "F.Cu")
-		(at 165 108.75)
+		(at 167 108.75)
 		(descr "https://www.amphenolrf.com/library/download/link/link_id/595984/parent/132289/")
 		(tags "SMA")
@@
 	(footprint "Capacitor_SMD:C_0603_1608Metric"
 		(layer "F.Cu")
-		(at 153.25 108.75)
+		(at 156.5 108.75)
 		(descr "Capacitor SMD 0603 (1608 Metric), square (rectangular) end terminal, IPC_7351 nominal, (Body size source: IPC-SM-782 page 76, https://www.pcb-3d.com/wordpress/wp-content/uploads/ipc-sm-782a_amendment_1_and_2.pdf), generated with kicad-footprint-generator")
 		(tags "capacitor")
@@
 	(footprint "Capacitor_Tantalum_SMD:CP_EIA-3528-15_AVX-H_HandSolder"
 		(layer "F.Cu")
-		(at 143.75 93.25)
+		(at 143.5 93.25)
 		(descr "Tantalum Capacitor SMD AVX-H (3528-15 Metric), IPC-7352 nominal, (Body size from: http://www.kemet.com/Lists/ProductCatalog/Attachments/253/KEM_TC101_STD.pdf), generated with kicad-footprint-generator")
 		(tags "capacitor tantalum")
@@
 	(footprint "Filter:Filter_Mini-Circuits_FV1206"
 		(layer "F.Cu")
-		(at 158 108.6775)
+		(at 160.75 108.6775)
 		(descr "Mini-Circuits Filter SMD 1206 https://ww2.minicircuits.com/case_style/FV1206.pdf")
 		(tags "Mini-Circuits Filter SMD 1206")
@@
 	(gr_line
 		(start 100.5 88.75)
-		(end 167.75 88.75)
+		(end 169.75 88.75)
 		(stroke
 			(width 0.05)
@@
 	)
 	(gr_line
-		(start 167.75 119.5)
+		(start 169.75 119.5)
 		(end 100.5 119.5)
 		(stroke
@@
 	)
 	(gr_line
-		(start 167.75 88.75)
-		(end 167.75 119.5)
+		(start 169.75 88.75)
+		(end 169.75 119.5)
 		(stroke
 			(width 0.05)
@@
 	)
 	(gr_text "RF-OUT"
-		(at 161 102.5 0)
+		(at 163.25 102.5 0)
 		(layer "F.SilkS")
 		(effects
@@
 	)
 	(segment
-		(start 156.3025 108.75)
-		(end 156.375 108.6775)
+		(start 159.0525 108.75)
+		(end 159.125 108.6775)
 		(width 0.2)
 		(layer "F.Cu")
@@
 	)
 	(segment
-		(start 156.375 108.6775)
-		(end 154.0975 108.6775)
+		(start 157.275 108.75)
+		(end 159.0525 108.75)
 		(width 0.75)
 		(layer "F.Cu")
@@
 	)
 	(segment
-		(start 154.0975 108.6775)
-		(end 154.025 108.75)
-		(width 0.2)
-		(layer "F.Cu")
-		(net 4)
-	)
-	(segment
 		(start 122.8 109.025)
 		(end 122.75 108.975)
@@
 	)
 	(segment
-		(start 152.475 108.75)
-		(end 146.5375 108.75)
+		(start 146.5375 108.75)
+		(end 155.725 108.75)
 		(width 0.75)
 		(layer "F.Cu")
@@
 	)
 	(segment
-		(start 159.625 108.6775)
-		(end 165.0725 108.6775)
+		(start 162.375 108.6775)
+		(end 166.9275 108.6775)
 		(width 0.75)
 		(layer "F.Cu")
@@
 	)
 	(segment
+		(start 166.9275 108.6775)
+		(end 167 108.75)
+		(width 0.2)
+		(layer "F.Cu")
+		(net 14)
+	)
+	(segment
 		(start 165.0725 108.6775)
 		(end 165.25 108.5)
@@
 		(polygon
 			(pts
-				(xy 100.5 111.25) (xy 100.5 119.5) (xy 115 119.5) (xy 115 111.25)
+				(xy 100.5 111) (xy 100.5 119.5) (xy 115 119.5) (xy 115 111)
 			)
 		)
@@
 		(layer "F.Cu")
 		(hatch edge 0.5)
-		(priority 4)
 		(connect_pads yes
 			(clearance 0)
@@
 		(polygon
 			(pts
-				(xy 157.5 110) (xy 158.5 110) (xy 158.5 110.75) (xy 157.5 110.75)
+				(xy 100.5 95) (xy 112.75 95) (xy 112.75 107) (xy 119.25 107) (xy 100.5 107)
 			)
 		)
@@
 		(layer "F.Cu")
 		(hatch edge 0.5)
+		(priority 11)
 		(connect_pads yes
 			(clearance 0)
@@
 		(polygon
 			(pts
-				(xy 100.5 94.75) (xy 112.75 94.75) (xy 112.75 107) (xy 119.25 107) (xy 100.5 107)
+				(xy 100.5 95) (xy 100.5 88.75) (xy 105.5 88.75) (xy 105.5 95)
 			)
 		)
@@
 		(layer "F.Cu")
 		(hatch edge 0.5)
-		(priority 11)
+		(priority 4)
 		(connect_pads yes
 			(clearance 0)
@@
 		(polygon
 			(pts
-				(xy 100.5 94.75) (xy 100.5 88.75) (xy 105.5 88.75) (xy 105.5 94.75)
+				(xy 154.75 111) (xy 169.75 111) (xy 169.75 119.5) (xy 154.75 119.5)
 			)
 		)
@@
 		(polygon
 			(pts
-				(xy 115 110.75) (xy 120 110.75) (xy 120 110.25) (xy 167.75 110.25) (xy 167.75 119.5) (xy 115 119.5)
+				(xy 115 110.75) (xy 120 110.75) (xy 120 110.25) (xy 154.75 110.25) (xy 154.75 119.5) (xy 115 119.5)
 			)
 		)
@@
 		(layer "F.Cu")
 		(hatch edge 0.5)
-		(priority 4)
+		(priority 13)
 		(connect_pads yes
 			(clearance 0)
@@
 		(polygon
 			(pts
-				(xy 157.5 106.75) (xy 158.5 106.75) (xy 158.5 107.5) (xy 157.5 107.5)
+				(xy 160.25 109.75) (xy 161.25 109.75) (xy 161.25 111) (xy 160.25 111)
 			)
 		)
@@
 		(layer "F.Cu")
 		(hatch edge 0.5)
+		(priority 12)
+		(connect_pads yes
+			(clearance 0)
+		)
+		(min_thickness 0.25)
+		(filled_areas_thickness no)
+		(fill yes
+			(thermal_gap 0.5)
+			(thermal_bridge_width 0.5)
+		)
+		(polygon
+			(pts
+				(xy 161.25 107.5) (xy 160.25 107.5) (xy 160.25 106.5) (xy 161.25 106.5)
+			)
+		)
+	)
+	(zone
+		(net 2)
+		(net_name "GND")
+		(layer "F.Cu")
+		(hatch edge 0.5)
 		(priority 8)
 		(connect_pads yes
@@
 		(polygon
 			(pts
-				(xy 143.5 107.25) (xy 143.5 88.75) (xy 167.75 88.75) (xy 167.75 107.25)
+				(xy 143.5 106.5) (xy 143.5 88.75) (xy 169.75 88.75) (xy 169.75 106.5)
 			)
 		)
@@
 		(priority 5)
 		(connect_pads yes
-			(clearance 0.5)
+			(clearance 0)
 		)
 		(min_thickness 0.25)
@@
 		(polygon
 			(pts
-				(xy 100.5 88.75) (xy 167.75 88.75) (xy 167.75 119.5) (xy 100.5 119.5)
+				(xy 100.5 88.75) (xy 169.75 88.75) (xy 169.75 119.5) (xy 100.5 119.5)
 			)
 		)
