File: PA-2W for sxceiver.kicad_pcb (KiCad board)
At the start: 2 copper layers, 72.8 x 30.5 mm, 40 parts, among them J1 SMA_RF IN, J2 SMA_RF OUT, J3 5Vcc input, U1 TQP3M9036, U2 TQP7M9106

Commit message: Add files via upload
Parts:
- removed FL1: LFCN-490, Filter:Filter_Mini-Circuits_FV1206
- added REF**: OSHW-Logo_5.7x6mm_SilkScreen, Symbol:OSHW-Logo_5.7x6mm_SilkScreen, F.Cu at (140.5, 114.8)
- moved J2 4.25 mm to (161.2, 108.8)
- moved H4 1.25 mm to (154.0, 98.2)
- moved H6 1.00 mm to (154.2, 116.0)
Connections:
- C12 pad 2: Net-(FL1-IN) -> Net-(J2-In)
- J2 pad 1: Net-(FL1-OUT) -> Net-(J2-In)
Routing:
- net Net-(J2-In): track 0.00 -> 5.13 mm
- net Net-(FL1-OUT): track 4.16 -> 0.00 mm
- net Net-(FL1-IN): track 2.23 -> 0.00 mm
- net GND: track 22.5 -> 20.4 mm, vias 14 -> 25
Other:
- board size 72.8 x 30.5 mm -> 68.5 x 30.8 mm
- board text added: "V1.1"
- board text added: "Z32IT"

Commit message: Add files via upload
Parts:
- removed C19: 1u, Capacitor_SMD:C_0805_2012Metric
- removed H5: MountingHole, MountingHole:MountingHole_2.2mm_M2_DIN965_Pad
- added FL1: LFCN-490, Filter:Filter_Mini-Circuits_FV1206, F.Cu at (160.0, 108.7)
- C16: footprint Capacitor_Tantalum_SMD:CP_EIA-6032-28_Kemet-C -> Capacitor_Tantalum_SMD:CP_EIA-3528-15_AVX-H_HandSolder
- C18: value 22u -> 47u; footprint Capacitor_Tantalum_SMD:CP_EIA-6032-28_Kemet-C -> Capacitor_Tantalum_SMD:CP_EIA-3528-15_AVX-H_HandSolder
- L1: footprint Inductor_SMD:L_0805_2012Metric -> Inductor_SMD:L_0603_1608Metric
- moved REF** 28.6 mm to (161.0, 94.8)
- moved C18 16.1 mm to (101.2, 99.5), turned to 180 degrees
- moved J2 4.75 mm to (165.9, 108.8)
- moved C17 2.14 mm to (114.0, 94.2), turned to 90 degrees
- moved H1 1.06 mm to (123.8, 99.0)
- moved H2 1.00 mm to (123.8, 116.0)
- moved H4 0.75 mm to (154.0, 99.0)
- moved C16 0.25 mm to (144.8, 93.2)
- turned C8 to 0 degrees
Connections:
- C12 pad 2: Net-(J2-In) -> Net-(FL1-IN)
- C14 pad 1: Net-(C13-Pad1) -> GND
- C14 pad 2: GND -> Net-(C13-Pad1)
- C18 pad 1: Net-(C13-Pad1) -> +5V
- C5 pad 1: Net-(C4-Pad2) -> Net-(C5-Pad1)
- C5 pad 2: Net-(C5-Pad2) -> Net-(C4-Pad1)
- C6 pad 1: Net-(C5-Pad2) -> Net-(C5-Pad1)
- C8 pad 1: GND -> Net-(C8-Pad1)
- C8 pad 2: Net-(C8-Pad2) -> GND
- C9 pad 1: GND -> Net-(U3-VBIAS)
- C9 pad 2: Net-(U3-VBIAS) -> GND
- J2 pad 1: Net-(J2-In) -> Net-(FL1-OUT)
- L1 pad 2: Net-(C4-Pad1) -> Net-(C4-Pad2)
- L2 pad 1: Net-(C8-Pad2) -> Net-(C8-Pad1)
- R1 pad 1: Net-(C4-Pad2) -> Net-(C4-Pad1)
- R1 pad 2: Net-(C5-Pad2) -> Net-(C5-Pad1)
- R2 pad 1: Net-(C5-Pad2) -> Net-(C5-Pad1)
- R3 pad 2: Net-(C8-Pad2) -> Net-(C8-Pad1)
- U1 pad 7: Net-(C4-Pad1) -> Net-(C4-Pad2)
Routing:
- net Net-(U1-VBIAS): track 11.8 -> 0.00 mm
- net (no net): track 0.00 -> 11.8 mm
- net Net-(C5-Pad2): track 7.39 -> 0.00 mm
- net Net-(C4-Pad1): track 5.24 -> 12.6 mm
- net Net-(J2-In): track 5.13 -> 0.00 mm
- net Net-(C8-Pad2): track 4.80 -> 0.00 mm
- net Net-(C8-Pad1): track 0.00 -> 4.80 mm
- net Net-(FL1-OUT): track 0.00 -> 4.31 mm
- net +5V: track 7.18 -> 10.7 mm
- net Net-(FL1-IN): track 0.00 -> 2.38 mm
- net GND: vias 25 -> 35
Other:
- board size 68.5 x 30.8 mm -> 73.2 x 30.8 mm
- board text added: "V1.2"
- board text removed: "V1.1"

Commit message: Add files via upload
Parts:
- moved C16 1.00 mm to (143.8, 93.2)
- moved C18 0.50 mm to (101.8, 99.5)
- turned C14 to 180 degrees
- turned C9 to 180 degrees
Connections:
- C9 pad 1: Net-(U3-VBIAS) -> Net-(U2-VBIAS)
- L2 pad 2: Net-(U3-I_REF) -> Net-(U2-I_REF)
- R4 pad 2: Net-(U3-VBIAS) -> Net-(U2-VBIAS)
- U2 pad 1: Net-(U1-VBIAS) -> Net-(U2-VBIAS)
- U2 pad 14: Net-(C10-Pad1) -> /RF_OUT/VCC
- U2 pad 15: Net-(C10-Pad1) -> /RF_OUT/VCC
- U2 pad 16: Net-(C10-Pad1) -> /RF_OUT/VCC
- U2 pad 18: Net-(U1-I_REF) -> Net-(U2-I_REF)
- U2 pad 4: Net-(C7-Pad1) -> /RF_IN
- U2 pad 5: Net-(C7-Pad1) -> /RF_IN
Routing:
- net Net-(C10-Pad1): track 13.9 -> 0.00 mm
- net /RF_OUT/VCC: track 0.00 -> 13.9 mm
- net Net-(U2-VBIAS): track 0.00 -> 11.8 mm
- net (no net): track 11.8 -> 0.00 mm
- net Net-(C7-Pad1): track 7.22 -> 0.00 mm
- net /RF_IN: track 0.00 -> 7.22 mm
- net Net-(U2-I_REF): track 0.00 -> 5.09 mm
- net Net-(U1-I_REF): track 5.09 -> 0.00 mm

Commit message: Add files via upload
Parts:
- removed the REF** at (161.0, 94.8)
- added REF**: OSHW-Logo2_7.3x6mm_Copper, Symbol:OSHW-Logo2_7.3x6mm_Copper, F.Cu at (163.8, 95.5)
- H1, H2, H3, H4, H6: footprint MountingHole:MountingHole_2.2mm_M2_DIN965_Pad -> MountingHole:MountingHole_2.7mm_M2.5_Pad_Via
- J1, J2: footprint PCM_SparkFun-Connector:SMA_Edge_6.3mm -> PCM_SparkFun-Connector:SMA_Edge_SMD
- moved J2 7.34 mm to (173.2, 108.8)
- moved J1 5.85 mm to (91.4, 109.0)
- moved H6 5.75 mm to (148.5, 116.0)
- moved H4 5.50 mm to (148.5, 99.0)
- moved C18 3.50 mm to (105.2, 99.5), turned to 0 degrees
- moved H1 2.50 mm to (126.2, 99.0)
- moved H2 2.48 mm to (126.2, 115.9)
- moved C9 1.50 mm to (131.5, 103.8), turned to 0 degrees
- moved C1 0.35 mm to (103.0, 109.0)
- moved U1 0.14 mm to (107.5, 109.2)
Connections:
- C4 pad 1: Net-(C4-Pad1) -> Net-(C4-Pad2)
- C4 pad 2: Net-(C4-Pad2) -> Net-(C4-Pad1)
- C5 pad 1: Net-(C5-Pad1) -> Net-(C4-Pad1)
- C5 pad 2: Net-(C4-Pad1) -> Net-(C5-Pad1)
- H1 pad 1: (no net) -> GND
- H2 pad 1: (no net) -> GND
- H3 pad 1: (no net) -> GND
- H4 pad 1: (no net) -> GND
- H6 pad 1: (no net) -> GND
Routing:
- net Net-(C4-Pad1): track 12.6 -> 5.10 mm
- net Net-(C5-Pad1): track 0.00 -> 7.45 mm
- net GND: track 20.4 -> 24.4 mm, vias 35 -> 46
- net Net-(J1-In): track 4.63 -> 2.72 mm
- net Net-(FL1-OUT): track 4.31 -> 3.55 mm
Other:
- board size 73.2 x 30.8 mm -> 82.8 x 30.8 mm
- board text added: "PA 2W"
- board text removed: "V1.2"

Commit message: Add files via upload
Other:
- board size 82.8 x 30.8 mm -> 82 x 30.8 mm
Changed lines of the file:
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@@
 	)
 	(gr_line
-		(start 91 88.75)
-		(end 173.75 88.75)
+		(start 91.25 88.75)
+		(end 173.24345 88.75)
 		(stroke
 			(width 0.05)
@@
 	)
 	(gr_line
-		(start 91 119.5)
-		(end 91 104.75)
+		(start 91.25 119.5)
+		(end 91.25 104.75)
 		(stroke
 			(width 0.05)
@@
 	)
 	(gr_line
-		(start 173.75 119.5)
-		(end 91 119.5)
+		(start 173.25 119.5)
+		(end 91.25 119.5)
 		(stroke
 			(width 0.05)
@@
 	)
 	(gr_line
-		(start 173.75 88.75)
-		(end 173.75 119.5)
+		(start 173.24345 88.75)
+		(end 173.24345 119.5)
 		(stroke
 			(width 0.05)
@@
 	)
 	(gr_line
-		(start 91 104.75)
-		(end 91 88.75)
+		(start 91.25 104.75)
+		(end 91.25 88.75)
 		(stroke
 			(width 0.05)
@@
 		(polygon
 			(pts
-				(xy 91 111.25) (xy 91 119.5) (xy 115 119.5) (xy 115 111.25)
+				(xy 91.25 111.25) (xy 91.25 119.5) (xy 115 119.5) (xy 115 111.25)
 			)
 		)
@@
 		(polygon
 			(pts
-				(xy 91 94.75) (xy 110.75 94.75) (xy 110.75 107) (xy 110.5 107) (xy 91 107)
+				(xy 91.25 94.75) (xy 110.75 94.75) (xy 110.75 107) (xy 110.5 107) (xy 91.25 107)
 			)
 		)
@@
 		(polygon
 			(pts
-				(xy 115 110.75) (xy 120 110.75) (xy 120 110.25) (xy 173.75 110.25) (xy 173.75 119.5) (xy 115 119.5)
+				(xy 115 110.75) (xy 120 110.75) (xy 120 110.25) (xy 173.25 110.25) (xy 173.25 119.5) (xy 115 119.5)
 			)
 		)
@@
 		(polygon
 			(pts
-				(xy 143.5 107) (xy 143.5 88.75) (xy 173.75 88.75) (xy 173.75 107)
+				(xy 143.5 107) (xy 143.5 88.75) (xy 173.25 88.75) (xy 173.25 107)
 			)
 		)
@@
 		(polygon
 			(pts
-				(xy 91 88.75) (xy 173.75 88.75) (xy 173.75 119.5) (xy 91 119.5)
+				(xy 91.25 88.75) (xy 173.25 88.75) (xy 173.25 119.5) (xy 91.25 119.5)
 			)
 		)

Commit message: Add files via upload
Parts:
- H1, H2, H3, H4, H6: footprint MountingHole:MountingHole_2.7mm_M2.5_Pad_Via -> MountingHole:MountingHole_2.2mm_M2_DIN965_Pad
- J1: value SMA_RF IN -> RF-in; footprint PCM_SparkFun-Connector:SMA_Edge_SMD -> Connector_Coaxial:SMA_Amphenol_132289_EdgeMount
- J2: value SMA_RF OUT -> RF-out; footprint PCM_SparkFun-Connector:SMA_Edge_SMD -> Connector_Coaxial:SMA_Amphenol_132289_EdgeMount
- moved J1 6.10 mm to (97.5, 109.0), turned to 180 degrees
- moved J2 6.00 mm to (167.2, 108.5), turned to 0 degrees
- moved REF** 4.43 mm to (159.5, 94.2)
- moved C3 3.50 mm to (112.5, 104.5)
- moved C2 3.25 mm to (112.5, 106.0)
- moved L1 2.25 mm to (111.8, 108.2)
- moved C4 1.75 mm to (114.2, 109.0), turned to 180 degrees
Connections:
- C4 pad 1: Net-(C4-Pad2) -> Net-(C4-Pad1)
- C4 pad 2: Net-(C4-Pad1) -> Net-(C4-Pad2)
- C5 pad 1: Net-(C4-Pad1) -> Net-(C5-Pad1)
- C5 pad 2: Net-(C5-Pad1) -> Net-(C4-Pad1)
- H1 pad 1: GND -> (no net)
- H2 pad 1: GND -> (no net)
- H3 pad 1: GND -> (no net)
- H4 pad 1: GND -> (no net)
- H6 pad 1: GND -> (no net)
- U1 pad 1: GND -> (no net)
- U1 pad 3: GND -> (no net)
- U1 pad 4: GND -> (no net)
- U1 pad 5: GND -> (no net)
- U1 pad 8: GND -> (no net)
Routing:
- net Net-(FL1-OUT): track 3.55 -> 6.20 mm
- net Net-(C13-Pad1): track 59.7 -> 62.2 mm
- net Net-(J1-In): track 2.72 -> 4.97 mm
- net Net-(C4-Pad1): track 5.10 -> 3.60 mm
- net GND: vias 46 -> 45
Other:
- board size 82 x 30.8 mm -> 75.8 x 30.8 mm

Commit message: Add files via upload
Parts:
- added R5: 10R, Resistor_SMD:R_0603_1608Metric, F.Cu at (138.8, 94.2)
- added R6: 10R, Resistor_SMD:R_0603_1608Metric, F.Cu at (130.8, 94.2)
- H1, H2, H3, H4, H6: footprint MountingHole:MountingHole_2.2mm_M2_DIN965_Pad -> MountingHole:MountingHole_2.7mm_M2.5_Pad_Via
- R3, R4: value 280R -> 270R
- moved C11 3.00 mm to (149.5, 109.8)
- moved L4 1.77 mm to (146.5, 109.0)
- moved C7 1.75 mm to (130.8, 109.8)
- moved J2 1.58 mm to (165.8, 109.0)
- moved C10 1.50 mm to (143.8, 109.8)
- moved H1 1.18 mm to (125.1, 99.0)
- moved R3 1.00 mm to (138.8, 97.8)
- moved R4 1.00 mm to (130.8, 97.8)
- moved H2 0.72 mm to (125.5, 115.9)
- moved C12 0.56 mm to (155.8, 109.0)
- moved R2 0.25 mm to (125.2, 109.0)
- moved FL1 0.25 mm to (160.0, 108.9)
- turned C5 to 180 degrees
Connections:
- H1 pad 1: (no net) -> GND
- H2 pad 1: (no net) -> GND
- H3 pad 1: (no net) -> GND
- H4 pad 1: (no net) -> GND
- H6 pad 1: (no net) -> GND
- R3 pad 1: Net-(C13-Pad1) -> Net-(R3-Pad1)
- R4 pad 1: Net-(C13-Pad1) -> Net-(R4-Pad1)
- U1 pad 1: (no net) -> GND
- U1 pad 3: (no net) -> GND
- U1 pad 4: (no net) -> GND
- U1 pad 5: (no net) -> GND
- U1 pad 8: (no net) -> GND
- U2 pad 27: (no net) -> GND
- U2 pad 28: (no net) -> GND
- U2 pad 29: (no net) -> GND
- U2 pad 30: (no net) -> GND
- U2 pad 31: (no net) -> GND
- U2 pad 32: (no net) -> GND
- U2 pad 33: (no net) -> GND
- U2 pad 34: (no net) -> GND
- U2 pad 35: (no net) -> GND
- U2 pad 36: (no net) -> GND
- U2 pad 37: (no net) -> GND
- U2 pad 38: (no net) -> GND
- U2 pad 39: (no net) -> GND
- U2 pad 40: (no net) -> GND
- U2 pad 41: (no net) -> GND
- U2 pad 42: (no net) -> GND
Routing:
- net GND: track 24.4 -> 6.41 mm, vias 45 -> 40
- net Net-(C13-Pad1): track 62.2 -> 56.9 mm
- net /RF_OUT/VCC: track 13.9 -> 11.3 mm
- net Net-(C11-Pad2): track 5.44 -> 7.69 mm
- net Net-(R4-Pad1): track 0.00 -> 1.85 mm
- net Net-(R3-Pad1): track 0.00 -> 1.85 mm
- net Net-(FL1-OUT): track 6.20 -> 4.41 mm
- net Net-(U2-VBIAS): track 11.8 -> 10.6 mm
- net Net-(C8-Pad1): track 4.80 -> 3.80 mm
- net Net-(FL1-IN): track 2.38 -> 1.88 mm
- added copper zone on F.Cu, net /RF_IN
- added copper zone on F.Cu, net /RF_OUT/VCC
Other:
- board size 75.8 x 30.8 mm -> 74 x 30.8 mm
