File: PA-2W for sxceiver.kicad_sch (KiCad schematic)
At the start: 40 parts, among them J1 SMA_RF IN, J2 SMA_RF OUT, J3 5Vcc input, U1 TQP3M9036, U3 TQP7M9106

Commit message: Add files via upload
Parts:
- removed FL1: LFCN-490, Filter:Filter_Mini-Circuits_FV1206, symbol RF_Filter:LFCN-490
Connections:
- net at C12.2: now also J2.1 (In)
Other:
- moved on the sheet: J2
Changed lines of the file:
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@@
 	(title_block
 		(title "SXceiver High Linearity Amplifier up to 2W")
-		(date "2026-03-15")
-		(rev "V1.0")
+		(date "2026-03-21")
+		(rev "V1.1")
 		(company "Z32IT")
 	)
@@
 	(wire
 		(pts
-			(xy 224.79 114.3) (xy 229.87 114.3)
-		)
-		(stroke
-			(width 0)
-			(type default)
-		)
-	)
-	(wire
-		(pts
 			(xy 74.93 55.88) (xy 90.17 55.88)
 		)
@@
 	(wire
 		(pts
-			(xy 250.19 114.3) (xy 254 114.3)
+			(xy 224.79 114.3) (xy 228.6 114.3)
 		)
 		(stroke
@@
 	(wire
 		(pts
-			(xy 259.08 119.38) (xy 259.08 123.19)
+			(xy 233.68 119.38) (xy 233.68 123.19)
 		)
 		(stroke
@@
 	(wire
 		(pts
-			(xy 240.03 124.46) (xy 240.03 128.27)
-		)
-		(stroke
-			(width 0)
-			(type default)
-		)
-	)
-	(wire
-		(pts
 			(xy 68.58 55.88) (xy 74.93 55.88)
 		)
@@
 	)
 	(symbol
-		(lib_id "PCM_4ms_Power-symbol:GND")
-		(at 240.03 128.27 0)
-		(unit 1)
-		(exclude_from_sim no)
-		(in_bom yes)
-		(on_board yes)
-		(dnp no)
-		(fields_autoplaced yes)
-		(property "Reference" "#PWR013"
-			(at 240.03 134.62 0)
-			(effects
-				(font
-					(size 1.27 1.27)
-				)
-				(hide yes)
-			)
-		)
-		(property "Value" "GND"
-			(at 240.03 133.35 0)
-			(effects
-				(font
-					(size 1.27 1.27)
-				)
-			)
-		)
-		(property "Footprint" ""
-			(at 240.03 128.27 0)
-			(effects
-				(font
-					(size 1.27 1.27)
-				)
-				(hide yes)
-			)
-		)
-		(property "Datasheet" ""
-			(at 240.03 128.27 0)
-			(effects
-				(font
-					(size 1.27 1.27)
-				)
-				(hide yes)
-			)
-		)
-		(property "Description" ""
-			(at 240.03 128.27 0)
-			(effects
-				(font
-					(size 1.27 1.27)
-				)
-				(hide yes)
-			)
-		)
-		(pin "1"
-		)
-		(instances
-			(project "LNA-2W"
-				(path "/9e841ece-bd19-4cb2-9a9c-7f7db9f00b2a"
-					(reference "#PWR013")
-					(unit 1)
-				)
-			)
-		)
-	)
-	(symbol
 		(lib_id "power:GND")
 		(at 80.01 71.12 0)
@@
 	)
 	(symbol
-		(lib_id "RF_Filter:LFCN-490")
-		(at 240.03 114.3 0)
-		(unit 1)
-		(exclude_from_sim no)
-		(in_bom yes)
-		(on_board yes)
-		(dnp no)
-		(fields_autoplaced yes)
-		(property "Reference" "FL1"
-			(at 240.03 101.6 0)
-			(effects
-				(font
-					(size 1.27 1.27)
-				)
-			)
-		)
-		(property "Value" "LFCN-490"
-			(at 240.03 104.14 0)
-			(effects
-				(font
-					(size 1.27 1.27)
-				)
-			)
-		)
-		(property "Footprint" "Filter:Filter_Mini-Circuits_FV1206"
-			(at 240.03 101.6 0)
-			(effects
-				(font
-					(size 1.27 1.27)
-				)
-				(hide yes)
-			)
-		)
-		(property "Datasheet" "https://www.minicircuits.com/pdfs/LFCN-490+.pdf"
-			(at 240.03 114.3 0)
-			(effects
-				(font
-					(size 1.27 1.27)
-				)
-				(hide yes)
-			)
-		)
-		(property "Description" "490MHz 50 Ohm Passive Low Pass Filter, FV1206"
-			(at 240.03 114.3 0)
-			(effects
-				(font
-					(size 1.27 1.27)
-				)
-				(hide yes)
-			)
-		)
-		(pin "1"
-		)
-		(pin "2"
-		)
-		(pin "3"
-		)
-		(pin "4"
-		)
-		(instances
-			(project ""
-				(path "/9e841ece-bd19-4cb2-9a9c-7f7db9f00b2a"
-					(reference "FL1")
-					(unit 1)
-				)
-			)
-		)
-	)
-	(symbol
 		(lib_id "Mechanical:MountingHole")
 		(at 264.16 26.67 0)
@@
 	(symbol
 		(lib_id "Connector:Conn_Coaxial")
-		(at 259.08 114.3 0)
+		(at 233.68 114.3 0)
 		(unit 1)
 		(exclude_from_sim no)
@@
 		(fields_autoplaced yes)
 		(property "Reference" "J2"
-			(at 262.89 113.3231 0)
+			(at 237.49 113.3231 0)
 			(effects
 				(font
@@
 		)
 		(property "Value" "SMA_RF OUT"
-			(at 262.89 115.8631 0)
+			(at 237.49 115.8631 0)
 			(effects
 				(font
@@
 		)
 		(property "Footprint" "PCM_SparkFun-Connector:SMA_Edge_6.3mm"
-			(at 259.08 114.3 0)
+			(at 233.68 114.3 0)
 			(effects
 				(font
@@
 		)
 		(property "Datasheet" "~"
-			(at 259.08 114.3 0)
+			(at 233.68 114.3 0)
 			(effects
 				(font
@@
 		)
 		(property "Description" "coaxial connector (BNC, SMA, SMB, SMC, Cinch/RCA, LEMO, ...)"
-			(at 259.08 114.3 0)
+			(at 233.68 114.3 0)
 			(effects
 				(font
@@
 	(symbol
 		(lib_id "PCM_4ms_Power-symbol:GND")
-		(at 259.08 123.19 0)
+		(at 233.68 123.19 0)
 		(unit 1)
 		(exclude_from_sim no)
@@
 		(fields_autoplaced yes)
 		(property "Reference" "#PWR04"
-			(at 259.08 129.54 0)
+			(at 233.68 129.54 0)
 			(effects
 				(font
@@
 		)
 		(property "Value" "GND"
-			(at 259.08 128.27 0)
+			(at 233.68 128.27 0)
 			(effects
 				(font
@@
 		)
 		(property "Footprint" ""
-			(at 259.08 123.19 0)
+			(at 233.68 123.19 0)
 			(effects
 				(font
@@
 		)
 		(property "Datasheet" ""
-			(at 259.08 123.19 0)
+			(at 233.68 123.19 0)
 			(effects
 				(font
@@
 		)
 		(property "Description" ""
-			(at 259.08 123.19 0)
+			(at 233.68 123.19 0)
 			(effects
 				(font

Commit message: Add files via upload
Parts:
- removed C19: 1u, Capacitor_SMD:C_0805_2012Metric, symbol Device:C_Small
- removed L1: 68n, Inductor_SMD:L_0805_2012Metric, symbol Device:L
- added FL1: LFCN-490, Filter:Filter_Mini-Circuits_FV1206, symbol RF_Filter:LFCN-490
- added L1: 68n, Inductor_SMD:L_0603_1608Metric, symbol Device:L_Small
- C1, C14, C2, C4, C5, C8, C9: DigiKey Part Number (none) -> 311-3599-1-ND; Manufacturer (none) -> YAGEO; Manufacturer Product Number (none) -> CC0603FRNPO9BN101
- C10, C6: DigiKey Part Number (none) -> 311-3347-1-ND; Manufacturer (none) -> YAGEO; Manufacturer Product Number (none) -> CC0603BRNPO9BN8R2
- C11: DigiKey Part Number (none) -> 311-3838-1-ND; Manufacturer (none) -> YAGEO; Manufacturer Product Number (none) -> CC0603BRNPO9BN6R8
- C12: DigiKey Part Number (none) -> 311-3350-1-ND; Manufacturer (none) -> YAGEO; Manufacturer Product Number (none) -> CC0603FRNPO9BN220
- C13, C15: DigiKey Part Number (none) -> 490-1451-1-ND; Manufacturer (none) -> Murata Electronics; Manufacturer Product Number (none) -> GRM1885C1H102JA01D
- C16: footprint Capacitor_Tantalum_SMD:CP_EIA-6032-28_Kemet-C -> Capacitor_Tantalum_SMD:CP_EIA-3528-15_AVX-H_HandSolder; DigiKey Part Number (none) -> 478-1682-1-ND; Manufacturer (none) -> KYOCERA AVX; Manufacturer Product Number (none) -> TAJB226K016RNJ
- C17: DigiKey Part Number (none) -> 311-4171-1-ND; Manufacturer (none) -> YAGEO; Manufacturer Product Number (none) -> CC0805FRNPO9BN220
- C18: value 22u -> 47u; footprint Capacitor_Tantalum_SMD:CP_EIA-6032-28_Kemet-C -> Capacitor_Tantalum_SMD:CP_EIA-3528-15_AVX-H_HandSolder; DigiKey Part Number (none) -> 478-1718-1-ND; Manufacturer (none) -> KYOCERA AVX; Manufacturer Product Number (none) -> TAJC476K016RNJ
- C3: DigiKey Part Number (none) -> 490-12330-1-ND; Manufacturer (none) -> Murata Electronics; Manufacturer Product Number (none) -> GRT188R61H105KE13D
- J1: DigiKey Part Number (none) -> CON-SMA-EDGE-S-ND; Manufacturer (none) -> RF Solutions; Manufacturer Product Number (none) -> CON-SMA-EDGE-S
- J2: DigiKey Part Number (none) -> CON-SMA-EDGE-S-ND; Manufacturer  (none) -> RF Solutions; Manufacturer Product Number (none) -> CON-SMA-EDGE-S
- J3: DigiKey Part Number (none) -> 277-12547-ND; Manufacturer (none) -> Phoenix Contact; Manufacturer Product Number (none) -> 5442206
- L2: Current (none) -> 600 mA; DigiKey Part Number (none) -> 490-15846-1-ND; Manufacturer (none) -> Murata Electronics; Manufacturer Product Number (none) -> LQW18AS68NG0ZD; Q min (none) -> 49.3
- L3: DigiKey Part Number (none) -> 535-AISC-1008HQ-18NG-TTR-ND; Manufacturer (none) -> Abracon LLC; Manufacturer Product Number (none) -> AISC-1008HQ-18NG-T; Q min (none) -> 62 @ 350 MHz
- L4: DigiKey Part Number (none) -> 490-LQW18AS4N7J00DCT-ND; Manufacturer (none) -> Murata Electronics; Manufacturer Product Number (none) -> LQW18AS4N7J00D
- L5: DigiKey Part Number (none) -> 240-2401-1-ND; Manufacturer (none) -> Laird-Signal Integrity Products; Manufacturer Product Number (none) -> LI1206H121R-10
- R1: DigiKey Part Number (none) -> 541-51.0HCT-ND; Manufacturer (none) -> Vishay Dale; Manufacturer Product Number (none) -> CRCW060351R0FKEA
- R2: DigiKey Part Number (none) -> 541-4.30HHCT-ND; Manufacturer (none) -> Vishay Dale; Manufacturer Product Number (none) -> CRCW06034R30FKEA
- R3, R4: DigiKey Part Number (none) -> 541-280HCT-ND; Manufacturer (none) -> Vishay Dale; Manufacturer Product Number (none) -> CRCW0603280RFKEA
- U1: Availability In Stock -> (none); Check_prices https://www.snapeda.com/parts/TQP3M9036/Qorvo/view-part/?re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 -> (none); Description_1 RF Amp Chip Single GP 2GHz 5.25V 8-Pin DFN EP T/R -> (none); DigiKey Part Number (none) -> 2312-TQP3M9036CT-ND; MANUFACTURER Qorvo -> (none); MAXIMUM_PACKAGE_HEIGHT 0.95mm -> (none); MF Qorvo -> (none); MP TQP3M9036 -> (none); Manufacturer (none) -> Qorvo; Manufacturer Product Number (none) -> TQP3M9036; PARTREV N/A -> (none); Package DFN-8 Qorvo -> (none); Price None -> (none); Purchase-URL https://www.snapeda.com/api/url_track_click_mouser/?unipart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 -> (none); STANDARD IPC-7351B -> (none); SnapEDA_Link https://www.snapeda.com/parts/TQP3M9036/Qorvo/view-part/?re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 -> (none)
- U3: Availability In Stock -> (none); Check_prices https://www.snapeda.com/parts/TQP7M9106/Qorvo/view-part/?re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 -> (none); Description_1 RF Amplifier IC CDMA, LTE, W-CDMA 50MHz ~ 1.5GHz 24-QFN (4x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 -> (none); DigiKey Part Number (none) -> 2312-TQP7M9106CT-ND; MANUFACTURER Qorvo -> (none); MAXIMUM_PACKAGE_HEIGHT 0.9 mm -> (none); MF Qorvo -> (none); MP TQP7M9106 -> (none); Manufacturer (none) -> Qorvo; Manufacturer Product Number (none) -> TQP7M9106; PARTREV Rev.D -> (none); Package QFN-24 Qorvo -> (none); Price None -> (none); SNAPEDA_PN TQP7M9106 -> (none); STANDARD IPC-7351B -> (none); SnapEDA_Link https://www.snapeda.com/parts/TQP7M9106/Qorvo/view-part/?re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 -> (none)
Connections:
- net +5V: now also C18.1
- net GND: now also C14.1, C8.2, C9.2, FL1.2 (GND), FL1.4 (GND); no longer C14.2, C8.1, C9.1
- net at C13.1, C15.1, C16.1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: now also C14.2, L1.1; no longer C14.1, C18.1
- net at R4.2, U3.1 (VBIAS): now also C9.1; no longer C9.2
- net at C6.1, R1.2, R2.1: now also C5.1; no longer C5.2
- net at L2.1, R3.2: now also C8.1; no longer C8.2
- net at C12.2: now also FL1.1 (IN); no longer J2.1 (In)
- net at C4.1: now also C5.2, R1.1; no longer U1.7
- new net: C4.2, L1.2, U1.7
- new net: FL1.3 (OUT), J2.1 (In)
Other:
- title: SXceiver High Linearity Amplifier up to 2W -> SXceiver Linear Amplifier up to 2W
- moved on the sheet: C18, J2

Commit message: Add files via upload
Parts:
- C7: DigiKey Part Number (none) -> 13-AC0603FRNPO9BN150CT-ND; Manufacturer (none) -> YAGEO; Manufacturer Product Number (none) -> AC0603FRNPO9BN150
- renumbered U3 to U2
Changed lines of the file:
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@@
 		(dnp no)
 		(fields_autoplaced yes)
-		(property "Reference" "U3"
+		(property "Reference" "U2"
 			(at 161.29 102.87 0)
 			(effects
@@
 			(project ""
 				(path "/9e841ece-bd19-4cb2-9a9c-7f7db9f00b2a"
-					(reference "U3")
+					(reference "U2")
 					(unit 1)
 				)
@@
 	)
 	(symbol
+		(lib_id "Device:C_Small")
+		(at 134.62 120.65 0)
+		(unit 1)
+		(exclude_from_sim no)
+		(in_bom yes)
+		(on_board yes)
+		(dnp no)
+		(property "Reference" "C7"
+			(at 129.286 120.65 90)
+			(effects
+				(font
+					(size 1.27 1.27)
+				)
+			)
+		)
+		(property "Value" "15p"
+			(at 131.572 120.65 90)
+			(effects
+				(font
+					(size 1.27 1.27)
+				)
+			)
+		)
+		(property "Footprint" "Capacitor_SMD:C_0603_1608Metric"
+			(at 134.62 120.65 0)
+			(effects
+				(font
+					(size 1.27 1.27)
+				)
+				(hide yes)
+			)
+		)
+		(property "Datasheet" "~"
+			(at 134.62 120.65 0)
+			(effects
+				(font
+					(size 1.27 1.27)
+				)
+				(hide yes)
+			)
+		)
+		(property "Description" "Unpolarized capacitor, small symbol"
+			(at 134.62 120.65 0)
+			(effects
+				(font
+					(size 1.27 1.27)
+				)
+				(hide yes)
+			)
+		)
+		(property "Manufacturer" "YAGEO"
+			(at 134.62 120.65 90)
+			(effects
+				(font
+					(size 1.27 1.27)
+				)
+				(hide yes)
+			)
+		)
+		(property "Manufacturer Product Number" "AC0603FRNPO9BN150"
+			(at 134.62 120.65 90)
+			(effects
+				(font
+					(size 1.27 1.27)
+				)
+				(hide yes)
+			)
+		)
+		(property "DigiKey Part Number" "13-AC0603FRNPO9BN150CT-ND"
+			(at 134.62 120.65 90)
+			(effects
+				(font
+					(size 1.27 1.27)
+				)
+				(hide yes)
+			)
+		)
+		(pin "1"
+		)
+		(pin "2"
+		)
+		(instances
+			(project "PA-2W for sxceiver"
+				(path "/9e841ece-bd19-4cb2-9a9c-7f7db9f00b2a"
+					(reference "C7")
+					(unit 1)
+				)
+			)
+		)
+	)
+	(symbol
 		(lib_id "Device:L_Ferrite_Small")
 		(at 90.17 59.69 0)
@@
 					(unit 1)
 				)
-			)
-		)
-	)
-	(symbol
-		(lib_id "Device:C_Small")
-		(at 134.62 120.65 0)
-		(unit 1)
-		(exclude_from_sim no)
-		(in_bom yes)
-		(on_board yes)
-		(dnp no)
-		(property "Reference" "C7"
-			(at 129.286 120.65 90)
-			(effects
-				(font
-					(size 1.27 1.27)
-				)
-			)
-		)
-		(property "Value" "15p"
-			(at 131.572 120.65 90)
-			(effects
-				(font
-					(size 1.27 1.27)
-				)
-			)
-		)
-		(property "Footprint" "Capacitor_SMD:C_0603_1608Metric"
-			(at 134.62 120.65 0)
-			(effects
-				(font
-					(size 1.27 1.27)
-				)
-				(hide yes)
-			)
-		)
-		(property "Datasheet" "~"
-			(at 134.62 120.65 0)
-			(effects
-				(font
-					(size 1.27 1.27)
-				)
-				(hide yes)
-			)
-		)
-		(property "Description" "Unpolarized capacitor, small symbol"
-			(at 134.62 120.65 0)
-			(effects
-				(font
-					(size 1.27 1.27)
-				)
-				(hide yes)
-			)
-		)
-		(pin "1"
-		)
-		(pin "2"
-		)
-		(instances
-			(project "LNA-2W"
-				(path "/9e841ece-bd19-4cb2-9a9c-7f7db9f00b2a"
-					(reference "C7")
-					(unit 1)
-				)

Commit message: Add files via upload
Parts:
- J1, J2: footprint PCM_SparkFun-Connector:SMA_Edge_6.3mm -> PCM_SparkFun-Connector:SMA_Edge_SMD
Other:
- title: SXceiver Linear Amplifier up to 2W -> PA 2W for HS without PA onboard
Changed lines of the file:
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@@
 	(paper "A4")
 	(title_block
-		(title "SXceiver Linear Amplifier up to 2W")
-		(date "2026-03-25")
-		(rev "V1.2")
+		(title "PA 2W for HS without PA onboard")
+		(date "2026-04-11")
+		(rev "V1.3")
 		(company "Z32IT")
 	)
@@
 			)
 		)
-		(property "Footprint" "PCM_SparkFun-Connector:SMA_Edge_6.3mm"
+		(property "Footprint" "PCM_SparkFun-Connector:SMA_Edge_SMD"
 			(at 260.35 114.3 0)
 			(effects
@@
 			)
 		)
-		(property "Footprint" "PCM_SparkFun-Connector:SMA_Edge_6.3mm"
+		(property "Footprint" "PCM_SparkFun-Connector:SMA_Edge_SMD"
 			(at 39.37 115.57 0)
 			(effects

Commit message: Add files via upload
Parts:
- removed J1: SMA_RF IN, PCM_SparkFun-Connector:SMA_Edge_SMD, symbol Connector:Conn_Coaxial
- removed J2: SMA_RF OUT, PCM_SparkFun-Connector:SMA_Edge_SMD, symbol Connector:Conn_Coaxial
- added J1: RF-in, Connector_Coaxial:SMA_Amphenol_132289_EdgeMount, symbol PCM_SparkFun-RF:SMA_EdgeMount_6.3mm
- added J2: RF-out, Connector_Coaxial:SMA_Amphenol_132289_EdgeMount, symbol PCM_SparkFun-RF:SMA_EdgeMount_6.3mm
Connections:
- net GND: now also J1.2 (Ext), J2.2 (Ext)
- net at FL1.3 (OUT): now also J2.1 (In)
- net at C1.2: now also J1.1 (In)
Changed lines of the file:
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@@
 	(title_block
 		(title "PA 2W for HS without PA onboard")
-		(date "2026-04-11")
-		(rev "V1.3")
+		(date "2026-04-12")
+		(rev "V1.4")
 		(company "Z32IT")
 	)
@@
 	)
 	(symbol
+		(lib_id "PCM_SparkFun-RF:SMA_EdgeMount_6.3mm")
+		(at 260.35 114.3 0)
+		(unit 1)
+		(exclude_from_sim no)
+		(in_bom yes)
+		(on_board yes)
+		(dnp no)
+		(property "Reference" "J2"
+			(at 264.16 115.8633 0)
+			(effects
+				(font
+					(size 1.27 1.27)
+				)
+				(justify left)
+			)
+		)
+		(property "Value" "RF-out"
+			(at 264.16 113.3233 0)
+			(effects
+				(font
+					(size 1.27 1.27)
+				)
+				(justify left)
+			)
+		)
+		(property "Footprint" "Connector_Coaxial:SMA_Amphenol_132289_EdgeMount"
+			(at 260.35 124.46 0)
+			(effects
+				(font
+					(size 1.27 1.27)
+				)
+				(hide yes)
+			)
+		)
+		(property "Datasheet" "https://cdn.sparkfun.com/assets/4/1/2/2/0/SMA-Connector.pdf"
+			(at 260.35 127 0)
+			(effects
+				(font
+					(size 1.27 1.27)
+				)
+				(hide yes)
+			)
+		)
+		(property "Description" "Not for new designs. Use 8mm variant. SMA PCB Edge Mount connector"
+			(at 260.35 129.54 0)
+			(effects
+				(font
+					(size 1.27 1.27)
+				)
+				(hide yes)
+			)
+		)
+		(property "PROD_ID" "CONN-08289"
+			(at 260.35 121.92 0)
+			(effects
+				(font
+					(size 1.27 1.27)
+				)
+				(hide yes)
+			)
+		)
+		(pin "1"
+		)
+		(pin "2"
+		)
+		(instances
+			(project "PA-2W for sxceiver"
+				(path "/9e841ece-bd19-4cb2-9a9c-7f7db9f00b2a"
+					(reference "J2")
+					(unit 1)
+				)
+			)
+		)
+	)
+	(symbol
 		(lib_id "RF_Filter:LFCN-490")
 		(at 240.03 114.3 0)
@@
 	)
 	(symbol
-		(lib_id "Connector:Conn_Coaxial")
-		(at 260.35 114.3 0)
-		(unit 1)
-		(exclude_from_sim no)
-		(in_bom yes)
-		(on_board yes)
-		(dnp no)
-		(fields_autoplaced yes)
-		(property "Reference" "J2"
-			(at 264.16 113.3231 0)
-			(effects
-				(font
-					(size 1.27 1.27)
-				)
-				(justify left)
-			)
-		)
-		(property "Value" "SMA_RF OUT"
-			(at 264.16 115.8631 0)
-			(effects
-				(font
-					(size 1.27 1.27)
-				)
-				(justify left)
-			)
-		)
-		(property "Footprint" "PCM_SparkFun-Connector:SMA_Edge_SMD"
-			(at 260.35 114.3 0)
-			(effects
-				(font
-					(size 1.27 1.27)
-				)
-				(hide yes)
-			)
-		)
-		(property "Datasheet" "~"
-			(at 260.35 114.3 0)
-			(effects
-				(font
-					(size 1.27 1.27)
-				)
-				(hide yes)
-			)
-		)
-		(property "Description" "coaxial connector (BNC, SMA, SMB, SMC, Cinch/RCA, LEMO, ...)"
-			(at 260.35 114.3 0)
-			(effects
-				(font
-					(size 1.27 1.27)
-				)
-				(hide yes)
-			)
-		)
-		(property "Manufacturer " "RF Solutions"
-			(at 260.35 114.3 0)
-			(effects
-				(font
-					(size 1.27 1.27)
-				)
-				(hide yes)
-			)
-		)
-		(property "Manufacturer Product Number" "CON-SMA-EDGE-S"
-			(at 260.35 114.3 0)
-			(effects
-				(font
-					(size 1.27 1.27)
-				)
-				(hide yes)
-			)
-		)
-		(property "DigiKey Part Number" "CON-SMA-EDGE-S-ND"
-			(at 260.35 114.3 0)
-			(effects
-				(font
-					(size 1.27 1.27)
-				)
-				(hide yes)
-			)
-		)
-		(pin "2"
-		)
-		(pin "1"
-		)
-		(instances
-			(project "LNA-2W"
-				(path "/9e841ece-bd19-4cb2-9a9c-7f7db9f00b2a"
-					(reference "J2")
-					(unit 1)
-				)
-			)
-		)
-	)
-	(symbol
 		(lib_id "Device:C_Small")
 		(at 54.61 115.57 270)
@@
 	)
 	(symbol
-		(lib_id "Connector:Conn_Coaxial")
+		(lib_id "PCM_SparkFun-RF:SMA_EdgeMount_6.3mm")
 		(at 39.37 115.57 0)
 		(mirror y)
@@
 			)
 		)
-		(property "Value" "SMA_RF IN"
+		(property "Value" "RF-in"
 			(at 35.56 114.5933 0)
 			(effects
@@
 			)
 		)
-		(property "Footprint" "PCM_SparkFun-Connector:SMA_Edge_SMD"
-			(at 39.37 115.57 0)
-			(effects
-				(font
-					(size 1.27 1.27)
-				)
-				(hide yes)
-			)
-		)
-		(property "Datasheet" "~"
-			(at 39.37 115.57 0)
+		(property "Footprint" "Connector_Coaxial:SMA_Amphenol_132289_EdgeMount"
+			(at 39.37 125.73 0)
 			(effects
 				(font
@@
 			)
 		)
-		(property "Description" "coaxial connector (BNC, SMA, SMB, SMC, Cinch/RCA, LEMO, ...)"
-			(at 39.37 115.57 0)
+		(property "Datasheet" "https://cdn.sparkfun.com/assets/4/1/2/2/0/SMA-Connector.pdf"
+			(at 39.37 128.27 0)
 			(effects
 				(font
@@
 			)
 		)
-		(property "Manufacturer" "RF Solutions"
-			(at 39.37 115.57 0)
+		(property "Description" "Not for new designs. Use 8mm variant. SMA PCB Edge Mount connector"
+			(at 39.37 130.81 0)
 			(effects
 				(font
@@
 			)
 		)
-		(property "Manufacturer Product Number" "CON-SMA-EDGE-S"
-			(at 39.37 115.57 0)
+		(property "PROD_ID" "CONN-08289"
+			(at 39.37 123.19 0)
 			(effects
 				(font
@@
 			)
 		)
-		(property "DigiKey Part Number" "CON-SMA-EDGE-S-ND"
-			(at 39.37 115.57 0)
-			(effects
-				(font
-					(size 1.27 1.27)
-				)
-				(hide yes)
-			)
+		(pin "1"
 		)
 		(pin "2"
 		)
-		(pin "1"
-		)
 		(instances
-			(project ""
+			(project "PA-2W for sxceiver"
 				(path "/9e841ece-bd19-4cb2-9a9c-7f7db9f00b2a"
 					(reference "J1")

Commit message: Add files via upload
Parts:
- added R5, R6: 10R, Resistor_SMD:R_0603_1608Metric, symbol Device:R_Small
- R3, R4: value 280R -> 270R
Connections:
- net at C13.1, C14.2, C15.1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: now also R5.1, R6.1; no longer R3.1, R4.1
- new net: R3.1, R5.2
- new net: R4.1, R6.2
